File: pcb/Dog Collar Light.sch (KiCad schematic (older format))
At the start: 25 parts, among them J1 AVR-ISP-6, Q1 MBT3904DW1T1G, U2 ATtiny84A-SSU

Commit message: Updated recommended switch to one that fits case better. It is much shorter so you can squish the case more to turn on/off.
Parts:
- S1: value 222PJVAAR -> 222JJVAAR
Changed lines of the file:
@@
 P 5600 2400
 F 0 "S1" H 5600 2747 60  0000 C CNN
-F 1 "222PJVAAR" H 5600 2641 60  0000 C CNN
+F 1 "222JJVAAR" H 5600 2641 60  0000 C CNN
 F 2 "mi-footprint:Switch_222PJVAAR" H 5800 2600 60  0001 L CNN
 F 3 "https://www.te.com/commerce/DocumentDelivery/DDEController?Action=srchrtrv&DocNm=1825910&DocType=Customer+Drawing&DocLang=English" H 5800 2700 60  0001 L CNN
